Commit message: i

File: description/camera.xacro (robot description, xacro)
@@ -2,27 +2,28 @@
 <robot xmlns:xacro="http://www.ros.org/wiki/xacro" >
     <joint name="camera_joint" type="fixed">
-        <parent link="chassis"/>
+        <parent link="base_link"/>
         <child link="camera_link"/>
-        <origin xyz="0.24 0 0.05" rpy="0 0.18 0"/>
+        <origin xyz="0.1125 0 0.0585" rpy="0 0 0"/>
     </joint>
     <link name="camera_link">
         <visual>
+            <origin xyz="0.013 0.015 0"/>
             <geometry>
-                <box size="0.010 0.03 0.03"/>
+                <box size="0.026 0.074 0.03"/>
             </geometry>
             <material name="black"/>
         </visual>
-        <visual>
-            <origin xyz="0 0 -0.05"/>
+        <!-- <visual>
+            <origin xyz="-0.013 -0.015 0"/>
             <geometry>
                 <cylinder radius="0.002" length="0.1"/>
             </geometry>
             <material name="black"/>
-        </visual>
+        </visual> -->
     </link>
     <joint name="camera_optical_joint" type="fixed">
         <parent link="camera_link"/>
         <child link="camera_link_optical"/>
-        <origin xyz="0 0 0" rpy="${-pi/2} 0 ${-pi/2}"/>
+        <origin xyz="0.02 0 0" rpy="${-pi/2} 0 ${-pi/2}"/>
     </joint>
     <link name="camera_link_optical"></link>

File: description/lidar.xacro (robot description, xacro)
@@ -2,22 +2,24 @@
 <robot xmlns:xacro="http://www.ros.org/wiki/xacro">
     <joint name="laser_joint" type="fixed">
-        <parent link="chassis"/>
+        <parent link="base_link"/>
         <child link="laser_frame"/>
-        <origin xyz="0.2 0.0 0.1" rpy="0.0 0.0 0.0"/>
+        <origin xyz="0.074 -0.04 0.0775" rpy="0.0 0.0 0.0"/>
     </joint>
     <link name="laser_frame">
         <visual>
+            <origin xyz="0 0 0.007" rpy="0 0 0"/>
             <geometry>
-                <cylinder radius="0.048" length="0.036"/>
+                <cylinder radius="0.017" length="0.014"/>
             </geometry>
             <material name="red"/>
         </visual>
         <collision>
+            <origin xyz="0 0 0.007" rpy="0 0 0"/>
             <geometry>
-                <cylinder radius="0.048" length="0.036"/>
+                <cylinder radius="0.017" length="0.014"/>
             </geometry>
         </collision>
-        <xacro:inertial_cylinder mass="0.1" length="0.036" radius="0.048">
-            <origin xyz="0 0 0" rpy="0 0 0"/>
+        <xacro:inertial_cylinder mass="0.08" length="0.014" radius="0.017">
+            <origin xyz="0 0 0.007" rpy="0 0 0"/>
         </xacro:inertial_cylinder>
     </link>

File: description/robot_core.xacro (robot description, xacro)
@@ -3,15 +3,15 @@
     <xacro:include filename="inertial_macros.xacro" />
     <xacro:property name="chassis_length" value="0.225"/>
-    <xacro:property name="chassis_width" value="0.15"/>
+    <xacro:property name="chassis_width" value="0.153"/>
     <xacro:property name="chassis_height" value="0.0975"/>
     <xacro:property name="chassis_mass" value="4.0"/>
     <xacro:property name="wheel_radius" value="0.048"/>
-    <xacro:property name="wheel_thickness" value="0.036"/>
+    <xacro:property name="wheel_thickness" value="0.04"/>
     <xacro:property name="wheel_mass" value="0.05"/>
     <xacro:property name="wheel_offset_x" value="0.073"/>
     <xacro:property name="wheel_offset_y" value="0.1"/>
     <xacro:property name="wheel_offset_z" value="0.02"/>
-    <xacro:property name="caster_wheel_radius" value="0.01"/>
-    <xacro:property name="caster_wheel_mass" value="0.01"/>
+    <xacro:property name="caster_wheel_radius" value="0.02"/>
+    <xacro:property name="caster_wheel_mass" value="0.02"/>
     <xacro:property name="caster_wheel_offset_x" value="0.073"/>
     <xacro:property name="caster_wheel_offset_z" value="${-wheel_radius + caster_wheel_radius}"/>
@@ -46,10 +46,10 @@
         <parent link="base_link"/>
         <child link="chassis"/>
-        <origin xyz="${-chassis_length/2} 0 0"/>
+        <origin xyz="0 0 -0.02"/>
     </joint>
     <link name="chassis">
         <!-- chassis visual -->
         <visual>
-            <origin xyz="${chassis_length/2} 0 ${chassis_height/2}"/>
+            <origin xyz="0 0 ${chassis_height/2}"/>
             <geometry>
                 <box size="${chassis_length} ${chassis_width} ${chassis_height}"/>
@@ -59,5 +59,5 @@
         <!-- chassis interact -->
         <collision>
-            <origin xyz="${chassis_length/2} 0 ${chassis_height/2}"/>
+            <origin xyz="0 0 ${chassis_height/2}"/>
             <geometry>
                 <box size="${chassis_length} ${chassis_width} ${chassis_height}"/>
@@ -66,5 +66,5 @@
         <!-- chassis phisical -->
         <xacro:inertial_box mass="2.0" x="${chassis_length}" y="${chassis_width}" z="${chassis_height}">
-            <origin xyz="${chassis_length/2} 0 ${chassis_height/2}" rpy="0 0 0"/>
+            <origin xyz="0 0 ${chassis_height/2}" rpy="0 0 0"/>
         </xacro:inertial_box>
     </link>
@@ -133,5 +133,5 @@
         <visual>
             <geometry>
-                <sphere radius="0.01"/>1
+                <sphere radius="${caster_wheel_radius}"/>1
             </geometry>
             <material name="blue"/>
@@ -139,8 +139,8 @@
         <collision>
             <geometry>
-                <sphere radius="0.01"/>
+                <sphere radius="${caster_wheel_radius}"/>
             </geometry>
         </collision>
-        <xacro:inertial_sphere mass="0.02" radius="0.01">
+        <xacro:inertial_sphere mass="${caster_wheel_mass}" radius="${caster_wheel_radius}">
             <origin xyz="0 0 0" rpy="0 0 0"/>
         </xacro:inertial_sphere>
