Commit message: i

File: description/crab_bot.urdf (robot description, URDF)
Before this commit: robot None, 6 links, 5 joints
Links:
- removed link chassis
- removed link left_wheel
- removed link right_wheel
- added link left_wheel_link; collision sphere radius=${wheel_radius}; visual cylinder length=${wheel_thickness} radius=${wheel_radius}
- added link right_wheel_link; collision sphere radius=${wheel_radius}; visual cylinder length=${wheel_thickness} radius=${wheel_radius}
- link base_link: geometry collision box size=${chassis_length} ${chassis_width} ${chassis_height}; visual box size=${chassis_length} ${chassis_width} ${chassis_height}
Joints:
- removed joint chassis_joint
- joint left_wheel_joint: axis 0 0 1 -> 0 1 0; child left_wheel -> left_wheel_link; origin xyz=${-wheel_offset_x} ${wheel_offset_y} 0 rpy=-${pi/2} 0 0 -> xyz=${-wheel_offset_x} ${wheel_offset_y} 0 rpy=0 0 0
- joint right_wheel_joint: axis 0 0 -1 -> 0 1 0; child right_wheel -> right_wheel_link; origin xyz=${-wheel_offset_x} ${-wheel_offset_y} 0 rpy=${pi/2} 0 0 -> xyz=${-wheel_offset_x} ${-wheel_offset_y} 0 rpy=0 0 0

File: description/gazebo_control.xacro (robot description, xacro)
@@ -16,9 +16,9 @@
             <max_wheel_acceleration>10.0</max_wheel_acceleration>
             <!-- Output -->
-            <odometry_frame>odom</odometry_frame>
-            <robot_base_frame>base_link</robot_base_frame>
             <publish_odom>true</publish_odom>
             <publish_odom_tf>true</publish_odom_tf>
             <publish_wheel_tf>true</publish_wheel_tf>
+            <odometry_frame>odom</odometry_frame>
+            <robot_base_frame>base_link</robot_base_frame>
         </plugin>
     </gazebo>

File: description/lidar.xacro (robot description, xacro)
@@ -1,5 +1,66 @@
 <?xml version="1.0"?>
 <robot xmlns:xacro="http://www.ros.org/wiki/xacro">
-    <joint name="laser_joint" type="fixed">
+    <!-- Lidar link -->
+    <link name="lidar_link">
+        <inertial>
+            <origin xyz="0 0 0" rpy="0 0 0"/>
+            <mass value="0.125"/>
+            <inertia ixx="0.001"  ixy="0"  ixz="0" iyy="0.001" iyz="0" izz="0.001" />
+        </inertial>
+        <collision>
+            <origin xyz="0 0 0" rpy="0 0 0"/>
+            <geometry>
+                <cylinder radius="0.017" length="0.014"/>
+            </geometry>
+        </collision>
+        <visual>
+            <origin xyz="0 0 0" rpy="0 0 0"/>
+            <geometry>
+                <cylinder radius="0.017" length="0.014"/>
+            </geometry>
+        </visual>
+    </link>
+    <!-- Lidar Joint -->
+    <joint name="lidar_joint" type="fixed">
+        <parent link="base_link"/>
+        <child link="lidar_link"/>
+        <origin xyz="0.074 -0.04 0.0845" rpy="0 0 0"/>
+    </joint>
+    <!-- Gazebo Plugin -->
+    <gazebo reference="lidar_link">
+        <sensor name="lidar" type="ray">
+            <always_on>true</always_on>
+            <visualize>true</visualize>
+            <update_rate>5</update_rate>
+            <ray>
+                <scan>
+                    <horizontal>
+                    <samples>360</samples>
+                    <resolution>1.000000</resolution>
+                    <min_angle>0.000000</min_angle>
+                    <max_angle>6.280000</max_angle>
+                    </horizontal>
+                </scan>
+                <range>
+                    <min>0.120000</min>
+                    <max>3.5</max>
+                    <resolution>0.015000</resolution>
+                </range>
+                <noise>
+                    <type>gaussian</type>
+                    <mean>0.0</mean>
+                    <stddev>0.01</stddev>
+                </noise>
+            </ray>
+            <plugin name="scan" filename="libgazebo_ros_ray_sensor.so">
+                <ros>
+                    <remapping>~/out:=scan</remapping>
+                </ros>
+                <output_type>sensor_msgs/LaserScan</output_type>
+                <frame_name>lidar_link</frame_name>
+            </plugin>
+        </sensor>
+    </gazebo>
+    <!-- <joint name="laser_joint" type="fixed">
         <parent link="base_link"/>
         <child link="laser_frame"/>
@@ -51,4 +112,4 @@
             </plugin>
         </sensor>
-    </gazebo>
+    </gazebo> -->
 </robot>

File: description/robot.urdf.xacro (robot description, xacro)
@@ -1,4 +1,4 @@
 <?xml version="1.0"?>
-<robot xmlns:xacro="http://www.ros.org/wiki/xacro"  name="robot">
+<robot xmlns:xacro="http://www.ros.org/wiki/xacro"  name="crab_bot">
     <xacro:include filename="robot_core.xacro" />
     <xacro:arg name="use_ros2_control" default="false"/>
@@ -10,5 +10,6 @@
     </xacro:unless>
     <xacro:include filename="lidar.xacro" />
-    <xacro:include filename="camera.xacro" />
+    <!-- <xacro:include filename="camera.xacro" /> -->
+    <xacro:include filename="dept_camera.xacro" />
     <xacro:include filename="imu.xacro" />
 </robot>
