Commit message: i

File: description/gazebo_control.xacro (robot description, xacro)
@@ -1,4 +1,4 @@
 <?xml version="1.0"?>
-<robot xmlns:xacro="http://www.ros.org/wiki/xacro"  name="robot">
+<robot xmlns:xacro="http://www.ros.org/wiki/xacro" >
     <gazebo>
         <plugin name="diff_drive" filename="libgazebo_ros_diff_drive.so">

File: description/robot.urdf.xacro (robot description, xacro)
@@ -2,5 +2,6 @@
 <robot xmlns:xacro="http://www.ros.org/wiki/xacro"  name="robot">
     <xacro:include filename="robot_core.xacro" />
-    <!-- <xacro:include filename="gazebo_control.xacro" /> -->
-    <xacro:include filename="ros2_control.xacro" />
+    <xacro:include filename="gazebo_control.xacro" />
+    <!-- <xacro:include filename="ros2_control.xacro" /> -->
+    <xacro:include filename="lidar.xacro" />
 </robot>

File: description/robot_core.xacro (robot description, xacro)
@@ -1,4 +1,4 @@
 <?xml version="1.0"?>
-<robot xmlns:xacro="http://www.ros.org/wiki/xacro"  name="robot">
+<robot xmlns:xacro="http://www.ros.org/wiki/xacro">
     <xacro:include filename="inertial_macros.xacro" />
     <material name="white">
@@ -13,4 +13,7 @@
     <material name="black">
         <color rgba="0 0 0 1"/>
+    </material>
+    <material name="red">
+        <color rgba="1 0 0 1"/>
     </material>
     <!-- Base link -->

File: description/ros2_control.xacro (robot description, xacro)
@@ -1,4 +1,4 @@
 <?xml version="1.0"?>
-<robot xmlns:xacro="http://www.ros.org/wiki/xacro"  name="robot">
+<robot xmlns:xacro="http://www.ros.org/wiki/xacro" >
     <ros2_control>
         <hardware>

Commit message: i

File: description/gazebo_control.xacro (robot description, xacro)
@@ -3,4 +3,5 @@
     <gazebo>
         <plugin name="diff_drive" filename="libgazebo_ros_diff_drive.so">
+        <!-- <plugin name="skid_steer_drive_controller" filename="libgazebo_ros_skid_steer_drive.so"> -->
             <ros>
                 <namespace>/demo</namespace>

File: description/imu.xacro (robot description, xacro)
@@ -6,10 +6,10 @@
         <visual>
             <geometry>
-                <box size="0.1 0.1 0.1"/>
+                <box size="0.02 0.02 0.02"/>
             </geometry>
         </visual>
         <collision>
             <geometry>
-                <box size="0.1 0.1 0.1"/>
+                <box size="0.02 0.02 0.02"/>
             </geometry>
         </collision>

File: description/robot.urdf.xacro (robot description, xacro)
@@ -2,5 +2,5 @@
 <robot xmlns:xacro="http://www.ros.org/wiki/xacro"  name="crab_bot">
     <xacro:include filename="robot_core.xacro" />
-    <xacro:arg name="use_ros2_control" default="false"/>
+    <xacro:arg name="use_ros2_control" default="true"/>
     <xacro:if value="$(arg use_ros2_control)">
         <xacro:include filename="ros2_control.xacro" />

File: description/robot_core.xacro (robot description, xacro)
@@ -65,5 +65,5 @@
         </collision>
         <!-- chassis phisical -->
-        <xacro:inertial_box mass="2.0" x="${chassis_length}" y="${chassis_width}" z="${chassis_height}">
+        <xacro:inertial_box mass="0.5" x="${chassis_length}" y="${chassis_width}" z="${chassis_height}">
             <origin xyz="0 0 ${chassis_height/2}" rpy="0 0 0"/>
         </xacro:inertial_box>
@@ -98,4 +98,29 @@
         <material>Gazebo/Blue</material>
     </gazebo>
+    <!-- <joint name="left_upper_wheel_joint" type="continuous">
+        <parent link="base_link"/>
+        <child link="left_upper_wheel"/>
+        <origin xyz="${wheel_offset_x} ${wheel_offset_y} 0" rpy="-${pi/2} 0 0"/>
+        <axis xyz="0 0 1"/>
+    </joint>
+    <link name="left_upper_wheel">
+        <visual>
+            <geometry>
+                <cylinder radius="${wheel_radius}" length="${wheel_thickness}"/>
+            </geometry>
+            <material name="blue"/>
+        </visual>
+        <collision>
+            <geometry>
+                <sphere radius="${wheel_radius}"/>
+            </geometry>
+        </collision>
+        <xacro:inertial_cylinder mass="${wheel_mass}" length="${wheel_thickness}" radius="${wheel_radius}">
+            <origin xyz="0 0 0" rpy="0 0 0"/>
+        </xacro:inertial_cylinder>
+    </link>
+    <gazebo reference="left_upper_wheel">
+        <material>Gazebo/Blue</material>
+    </gazebo> -->
     <!-- Right wheel link -->
     <joint name="right_wheel_joint" type="continuous">
@@ -124,4 +149,29 @@
         <material>Gazebo/Blue</material>
     </gazebo>
+    <!-- <joint name="right_upper_wheel_joint" type="continuous">
+        <parent link="base_link"/>
+        <child link="right_upper_wheel"/>
+        <origin xyz="${wheel_offset_x} ${-wheel_offset_y} 0" rpy="${pi/2} 0 0"/>
+        <axis xyz="0 0 -1"/>
+    </joint>
+    <link name="right_upper_wheel">
+        <visual>
+            <geometry>
+                <cylinder radius="${wheel_radius}" length="${wheel_thickness}"/>
+            </geometry>
+            <material name="blue"/>
+        </visual>
+        <collision>
+            <geometry>
+                <sphere radius="${wheel_radius}"/>
+            </geometry>
+        </collision>
+        <xacro:inertial_cylinder mass="${wheel_mass}" length="${wheel_thickness}" radius="${wheel_radius}">
+            <origin xyz="0 0 0" rpy="0 0 0"/>
+        </xacro:inertial_cylinder>
+    </link>
+    <gazebo reference="right_upper_wheel">
+        <material>Gazebo/Blue</material>
+    </gazebo> -->
     <!-- Caster wheel link -->
     <joint name="caster_wheel_joint" type="fixed">

File: description/ros2_control.xacro (robot description, xacro)
@@ -13,4 +13,12 @@
             <state_interface name="position"/>
         </joint>
+        <!-- <joint name="left_upper_wheel_joint" >
+            <command_interface name="velocity">
+                <param name="min">-10</param>
+                <param name="max">10</param>
+            </command_interface>
+            <state_interface name="velocity"/>
+            <state_interface name="position"/>
+        </joint> -->
         <joint name="right_wheel_joint" >
             <command_interface name="velocity">
@@ -21,4 +29,12 @@
             <state_interface name="position"/>
         </joint>
+        <!-- <joint name="right_wheel_joint" >
+            <command_interface name="velocity">
+                <param name="min">-10</param>
+                <param name="max">10</param>
+            </command_interface>
+            <state_interface name="velocity"/>
+            <state_interface name="position"/>
+        </joint> -->
     </ros2_control>
     <gazebo>

Commit message: i

File: description/gazebo_control.xacro (robot description, xacro)
@@ -5,15 +5,22 @@
         <!-- <plugin name="skid_steer_drive_controller" filename="libgazebo_ros_skid_steer_drive.so"> -->
             <ros>
-                <namespace>/demo</namespace>
+                <namespace>/gz_ctrl</namespace>
             </ros>
+            <!-- Number of wheel pairs -->
+            <num_wheel_pairs>2</num_wheel_pairs>
             <!-- Wheels -->
-            <left_joint>left_wheel_joint</left_joint>
-            <right_joint>right_wheel_joint</right_joint>
+            <left_joint>front_left_wheel_joint</left_joint>
+            <right_joint>front_right_wheel_joint</right_joint>
+            <left_joint>rear_left_wheel_joint</left_joint>
+            <right_joint>rear_right_wheel_joint</right_joint>
             <!-- Kinematic -->
             <wheel_separation>0.2</wheel_separation>
+            <wheel_separation>0.2</wheel_separation>
+            <wheel_diameter>0.096</wheel_diameter>
             <wheel_diameter>0.096</wheel_diameter>
             <!-- Limits -->
             <max_wheel_torque>200</max_wheel_torque>
             <max_wheel_acceleration>10.0</max_wheel_acceleration>
+            <command_topic>cmd_vel</command_topic>
             <!-- Output -->
             <publish_odom>true</publish_odom>

File: description/lidar.xacro (robot description, xacro)
@@ -31,5 +31,5 @@
         <sensor name="lidar" type="ray">
             <always_on>true</always_on>
-            <visualize>true</visualize>
+            <visualize>false</visualize>
             <update_rate>5</update_rate>
             <ray>

File: description/robot.urdf.xacro (robot description, xacro)
@@ -6,5 +6,4 @@
     <xacro:if value="$(arg use_ros2_control)">
         <xacro:include filename="ros2_control_4wd.xacro" />
-        <!-- <xacro:include filename="ros2_control.xacro" /> -->
     </xacro:if>
     <xacro:unless value="$(arg use_ros2_control)">

File: description/robot_core_4wd.xacro (robot description, xacro)
@@ -8,12 +8,9 @@
     <xacro:property name="wheel_radius" value="0.048"/>
     <xacro:property name="wheel_thickness" value="0.04"/>
-    <xacro:property name="wheel_mass" value="0.05"/>
+    <xacro:property name="wheel_mass" value="0.1"/>
+    <xacro:property name="wheel_separation" value="0.205"/>
     <xacro:property name="wheel_offset_x" value="0.073"/>
-    <xacro:property name="wheel_offset_y" value="0.1"/>
-    <xacro:property name="wheel_offset_z" value="0.02"/>
-    <xacro:property name="caster_wheel_radius" value="0.02"/>
-    <xacro:property name="caster_wheel_mass" value="0.02"/>
-    <xacro:property name="caster_wheel_offset_x" value="0.073"/>
-    <xacro:property name="caster_wheel_offset_z" value="${-wheel_radius + caster_wheel_radius}"/>
+    <xacro:property name="wheel_offset_y" value="${wheel_separation/2}"/>
+    <xacro:property name="chassis_offset_z" value="0.02"/>
     <material name="white">
         <color rgba="1 1 1 1"/>
@@ -46,5 +43,5 @@
         <parent link="base_link"/>
         <child link="chassis"/>
-        <origin xyz="0 0 -0.02"/>
+        <origin xyz="0 0 ${-chassis_offset_z}"/>
     </joint>
     <link name="chassis">
@@ -97,4 +94,6 @@
     <gazebo reference="rear_left_wheel">
         <material>Gazebo/Blue</material>
+        <mu1 value="1.0"/>
+        <mu2 value="0.5"/>
     </gazebo>
     <!-- FRONT LEFT WHEEL LINK -->
@@ -123,4 +122,6 @@
     <gazebo reference="front_left_wheel">
         <material>Gazebo/Blue</material>
+        <mu1 value="1.0"/>
+        <mu2 value="0.5"/>
     </gazebo>
     <!-- REAR RIGHT WHEEL LINK -->
@@ -149,4 +150,6 @@
     <gazebo reference="rear_right_wheel">
         <material>Gazebo/Blue</material>
+        <mu1 value="1.0"/>
+        <mu2 value="0.5"/>
     </gazebo>
     <!-- FRONT RIGHT WHEEL LINK -->
@@ -175,31 +178,6 @@
     <gazebo reference="front_right_wheel">
         <material>Gazebo/Blue</material>
-    </gazebo>
-    <!-- CASTER WHEEL LINK -->
-    <joint name="caster_wheel_joint" type="fixed">
-        <parent link="base_link"/>
-        <child link="caster_wheel"/>
-        <origin xyz="${caster_wheel_offset_x} 0 ${caster_wheel_offset_z}"/>
-    </joint>
-    <link name="caster_wheel">
-        <visual>
-            <geometry>
-                <sphere radius="${caster_wheel_radius}"/>1
-            </geometry>
-            <material name="blue"/>
-        </visual>
-        <collision>
-            <geometry>
-                <sphere radius="${caster_wheel_radius}"/>
-            </geometry>
-        </collision>
-        <xacro:inertial_sphere mass="${caster_wheel_mass}" radius="${caster_wheel_radius}">
-            <origin xyz="0 0 0" rpy="0 0 0"/>
-        </xacro:inertial_sphere>
-    </link>
-    <gazebo reference="caster_wheel">
-        <material>Gazebo/Blue</material>
-        <mu1 value="0.001"/>
-        <mu2 value="0.001"/>
+        <mu1 value="1.0"/>
+        <mu2 value="0.5"/>
     </gazebo>
 </robot>
