Commit message: i

File: description/gazebo_control.xacro (robot description, xacro)
@@ -15,6 +15,6 @@
             <right_joint>rear_right_wheel_joint</right_joint>
             <!-- Kinematic -->
-            <wheel_separation>0.2</wheel_separation>
-            <wheel_separation>0.2</wheel_separation>
+            <wheel_separation>0.205</wheel_separation>
+            <wheel_separation>0.205</wheel_separation>
             <wheel_diameter>0.096</wheel_diameter>
             <wheel_diameter>0.096</wheel_diameter>

File: description/robot.urdf.xacro (robot description, xacro)
@@ -1,9 +1,14 @@
 <?xml version="1.0"?>
 <robot xmlns:xacro="http://www.ros.org/wiki/xacro"  name="crab_bot">
-    <!-- <xacro:include filename="robot_core.xacro" /> -->
-    <xacro:include filename="robot_core_4wd.xacro" />
+    <xacro:include filename="robot_core.xacro" />
     <xacro:arg name="use_ros2_control" default="false"/>
+    <xacro:arg name="use_sim" default="true"/>
     <xacro:if value="$(arg use_ros2_control)">
-        <xacro:include filename="ros2_control_4wd.xacro" />
+        <xacro:if value="$(arg use_sim)">
+            <xacro:include filename="ros2_control.simulation.xacro" />
+        </xacro:if>
+        <xacro:unless value="$(arg use_sim)">
+            <xacro:include filename="ros2_control.hardware.xacro" />
+        </xacro:unless>
     </xacro:if>
     <xacro:unless value="$(arg use_ros2_control)">

File: description/robot_core.xacro (robot description, xacro)
@@ -8,12 +8,9 @@
     <xacro:property name="wheel_radius" value="0.048"/>
     <xacro:property name="wheel_thickness" value="0.04"/>
-    <xacro:property name="wheel_mass" value="0.05"/>
+    <xacro:property name="wheel_mass" value="0.1"/>
+    <xacro:property name="wheel_separation" value="0.205"/>
     <xacro:property name="wheel_offset_x" value="0.073"/>
-    <xacro:property name="wheel_offset_y" value="0.1"/>
-    <xacro:property name="wheel_offset_z" value="0.02"/>
-    <xacro:property name="caster_wheel_radius" value="0.02"/>
-    <xacro:property name="caster_wheel_mass" value="0.02"/>
-    <xacro:property name="caster_wheel_offset_x" value="0.073"/>
-    <xacro:property name="caster_wheel_offset_z" value="${-wheel_radius + caster_wheel_radius}"/>
+    <xacro:property name="wheel_offset_y" value="${wheel_separation/2}"/>
+    <xacro:property name="chassis_offset_z" value="0.02"/>
     <material name="white">
         <color rgba="1 1 1 1"/>
@@ -31,5 +28,5 @@
         <color rgba="1 0 0 1"/>
     </material>
-    <!-- Base link -->
+    <!-- BASE LINK -->
     <link name="base_link">
     </link>
@@ -42,9 +39,9 @@
     <link name="base_footprint">
     </link>
-    <!-- Chassis link -->
+    <!-- CHASSIS LINK -->
     <joint name="chassis_joint" type="fixed">
         <parent link="base_link"/>
         <child link="chassis"/>
-        <origin xyz="0 0 -0.02"/>
+        <origin xyz="0 0 ${-chassis_offset_z}"/>
     </joint>
     <link name="chassis">
@@ -72,12 +69,12 @@
         <material>Gazebo/White</material>
     </gazebo>
-    <!-- Left wheel link -->
-    <joint name="left_wheel_joint" type="continuous">
+    <!-- REAR LEFT WHEEL LINK -->
+    <joint name="rear_left_wheel_joint" type="continuous">
         <parent link="base_link"/>
-        <child link="left_wheel"/>
+        <child link="rear_left_wheel"/>
         <origin xyz="${-wheel_offset_x} ${wheel_offset_y} 0" rpy="-${pi/2} 0 0"/>
         <axis xyz="0 0 1"/>
     </joint>
-    <link name="left_wheel">
+    <link name="rear_left_wheel">
         <visual>
             <geometry>
@@ -95,14 +92,17 @@
         </xacro:inertial_cylinder>
     </link>
-    <gazebo reference="left_wheel">
+    <gazebo reference="rear_left_wheel">
         <material>Gazebo/Blue</material>
+        <mu1 value="1.0"/>
+        <mu2 value="0.5"/>
     </gazebo>
-    <!-- <joint name="left_upper_wheel_joint" type="continuous">
+    <!-- FRONT LEFT WHEEL LINK -->
+    <joint name="front_left_wheel_joint" type="continuous">
         <parent link="base_link"/>
-        <child link="left_upper_wheel"/>
+        <child link="front_left_wheel"/>
         <origin xyz="${wheel_offset_x} ${wheel_offset_y} 0" rpy="-${pi/2} 0 0"/>
         <axis xyz="0 0 1"/>
     </joint>
-    <link name="left_upper_wheel">
+    <link name="front_left_wheel">
         <visual>
             <geometry>
@@ -120,15 +120,17 @@
         </xacro:inertial_cylinder>
     </link>
-    <gazebo reference="left_upper_wheel">
+    <gazebo reference="front_left_wheel">
         <material>Gazebo/Blue</material>
-    </gazebo> -->
-    <!-- Right wheel link -->
-    <joint name="right_wheel_joint" type="continuous">
+        <mu1 value="1.0"/>
+        <mu2 value="0.5"/>
+    </gazebo>
+    <!-- REAR RIGHT WHEEL LINK -->
+    <joint name="rear_right_wheel_joint" type="continuous">
         <parent link="base_link"/>
-        <child link="right_wheel"/>
+        <child link="rear_right_wheel"/>
         <origin xyz="${-wheel_offset_x} ${-wheel_offset_y} 0" rpy="${pi/2} 0 0"/>
         <axis xyz="0 0 -1"/>
     </joint>
-    <link name="right_wheel">
+    <link name="rear_right_wheel">
         <visual>
             <geometry>
@@ -146,14 +148,17 @@
         </xacro:inertial_cylinder>
     </link>
-    <gazebo reference="right_wheel">
+    <gazebo reference="rear_right_wheel">
         <material>Gazebo/Blue</material>
+        <mu1 value="1.0"/>
+        <mu2 value="0.5"/>
     </gazebo>
-    <!-- <joint name="right_upper_wheel_joint" type="continuous">
+    <!-- FRONT RIGHT WHEEL LINK -->
+    <joint name="front_right_wheel_joint" type="continuous">
         <parent link="base_link"/>
-        <child link="right_upper_wheel"/>
+        <child link="front_right_wheel"/>
         <origin xyz="${wheel_offset_x} ${-wheel_offset_y} 0" rpy="${pi/2} 0 0"/>
         <axis xyz="0 0 -1"/>
     </joint>
-    <link name="right_upper_wheel">
+    <link name="front_right_wheel">
         <visual>
             <geometry>
@@ -171,33 +176,8 @@
         </xacro:inertial_cylinder>
     </link>
-    <gazebo reference="right_upper_wheel">
+    <gazebo reference="front_right_wheel">
         <material>Gazebo/Blue</material>
-    </gazebo> -->
-    <!-- Caster wheel link -->
-    <joint name="caster_wheel_joint" type="fixed">
-        <parent link="base_link"/>
-        <child link="caster_wheel"/>
-        <origin xyz="${caster_wheel_offset_x} 0 ${caster_wheel_offset_z}"/>
-    </joint>
-    <link name="caster_wheel">
-        <visual>
-            <geometry>
-                <sphere radius="${caster_wheel_radius}"/>1
-            </geometry>
-            <material name="blue"/>
-        </visual>
-        <collision>
-            <geometry>
-                <sphere radius="${caster_wheel_radius}"/>
-            </geometry>
-        </collision>
-        <xacro:inertial_sphere mass="${caster_wheel_mass}" radius="${caster_wheel_radius}">
-            <origin xyz="0 0 0" rpy="0 0 0"/>
-        </xacro:inertial_sphere>
-    </link>
-    <gazebo reference="caster_wheel">
-        <material>Gazebo/Blue</material>
-        <mu1 value="0.001"/>
-        <mu2 value="0.001"/>
+        <mu1 value="1.0"/>
+        <mu2 value="0.5"/>
     </gazebo>
 </robot>

File: description/robot_core_2wd.xacro (robot description, xacro)
@@ -8,9 +8,12 @@
     <xacro:property name="wheel_radius" value="0.048"/>
     <xacro:property name="wheel_thickness" value="0.04"/>
-    <xacro:property name="wheel_mass" value="0.1"/>
-    <xacro:property name="wheel_separation" value="0.205"/>
+    <xacro:property name="wheel_mass" value="0.05"/>
     <xacro:property name="wheel_offset_x" value="0.073"/>
-    <xacro:property name="wheel_offset_y" value="${wheel_separation/2}"/>
-    <xacro:property name="chassis_offset_z" value="0.02"/>
+    <xacro:property name="wheel_offset_y" value="0.1"/>
+    <xacro:property name="wheel_offset_z" value="0.02"/>
+    <xacro:property name="caster_wheel_radius" value="0.02"/>
+    <xacro:property name="caster_wheel_mass" value="0.02"/>
+    <xacro:property name="caster_wheel_offset_x" value="0.073"/>
+    <xacro:property name="caster_wheel_offset_z" value="${-wheel_radius + caster_wheel_radius}"/>
     <material name="white">
         <color rgba="1 1 1 1"/>
@@ -28,5 +31,5 @@
         <color rgba="1 0 0 1"/>
     </material>
-    <!-- BASE LINK -->
+    <!-- Base link -->
     <link name="base_link">
     </link>
@@ -39,9 +42,9 @@
     <link name="base_footprint">
     </link>
-    <!-- CHASSIS LINK -->
+    <!-- Chassis link -->
     <joint name="chassis_joint" type="fixed">
         <parent link="base_link"/>
         <child link="chassis"/>
-        <origin xyz="0 0 ${-chassis_offset_z}"/>
+        <origin xyz="0 0 -0.02"/>
     </joint>
     <link name="chassis">
@@ -69,115 +72,132 @@
         <material>Gazebo/White</material>
     </gazebo>
-    <!-- REAR LEFT WHEEL LINK -->
-    <joint name="rear_left_wheel_joint" type="continuous">
-        <parent link="base_link"/>
-        <child link="rear_left_wheel"/>
+    <!-- Left wheel link -->
+    <joint name="left_wheel_joint" type="continuous">
+        <parent link="base_link"/>
+        <child link="left_wheel"/>
         <origin xyz="${-wheel_offset_x} ${wheel_offset_y} 0" rpy="-${pi/2} 0 0"/>
         <axis xyz="0 0 1"/>
     </joint>
-    <link name="rear_left_wheel">
-        <visual>
-            <geometry>
-                <cylinder radius="${wheel_radius}" length="${wheel_thickness}"/>
-            </geometry>
-            <material name="blue"/>
-        </visual>
-        <collision>
-            <geometry>
-                <sphere radius="${wheel_radius}"/>
-            </geometry>
-        </collision>
-        <xacro:inertial_cylinder mass="${wheel_mass}" length="${wheel_thickness}" radius="${wheel_radius}">
-            <origin xyz="0 0 0" rpy="0 0 0"/>
-        </xacro:inertial_cylinder>
-    </link>
-    <gazebo reference="rear_left_wheel">
-        <material>Gazebo/Blue</material>
-        <mu1 value="1.0"/>
-        <mu2 value="0.5"/>
-    </gazebo>
-    <!-- FRONT LEFT WHEEL LINK -->
-    <joint name="front_left_wheel_joint" type="continuous">
-        <parent link="base_link"/>
-        <child link="front_left_wheel"/>
+    <link name="left_wheel">
+        <visual>
+            <geometry>
+                <cylinder radius="${wheel_radius}" length="${wheel_thickness}"/>
+            </geometry>
+            <material name="blue"/>
+        </visual>
+        <collision>
+            <geometry>
+                <sphere radius="${wheel_radius}"/>
+            </geometry>
+        </collision>
+        <xacro:inertial_cylinder mass="${wheel_mass}" length="${wheel_thickness}" radius="${wheel_radius}">
+            <origin xyz="0 0 0" rpy="0 0 0"/>
+        </xacro:inertial_cylinder>
+    </link>
+    <gazebo reference="left_wheel">
+        <material>Gazebo/Blue</material>
+    </gazebo>
+    <!-- <joint name="left_upper_wheel_joint" type="continuous">
+        <parent link="base_link"/>
+        <child link="left_upper_wheel"/>
         <origin xyz="${wheel_offset_x} ${wheel_offset_y} 0" rpy="-${pi/2} 0 0"/>
         <axis xyz="0 0 1"/>
     </joint>
-    <link name="front_left_wheel">
-        <visual>
-            <geometry>
-                <cylinder radius="${wheel_radius}" length="${wheel_thickness}"/>
-            </geometry>
-            <material name="blue"/>
-        </visual>
-        <collision>
-            <geometry>
-                <sphere radius="${wheel_radius}"/>
-            </geometry>
-        </collision>
-        <xacro:inertial_cylinder mass="${wheel_mass}" length="${wheel_thickness}" radius="${wheel_radius}">
-            <origin xyz="0 0 0" rpy="0 0 0"/>
-        </xacro:inertial_cylinder>
-    </link>
-    <gazebo reference="front_left_wheel">
-        <material>Gazebo/Blue</material>
-        <mu1 value="1.0"/>
-        <mu2 value="0.5"/>
-    </gazebo>
-    <!-- REAR RIGHT WHEEL LINK -->
-    <joint name="rear_right_wheel_joint" type="continuous">
-        <parent link="base_link"/>
-        <child link="rear_right_wheel"/>
+    <link name="left_upper_wheel">
+        <visual>
+            <geometry>
+                <cylinder radius="${wheel_radius}" length="${wheel_thickness}"/>
+            </geometry>
+            <material name="blue"/>
+        </visual>
+        <collision>
+            <geometry>
+                <sphere radius="${wheel_radius}"/>
+            </geometry>
+        </collision>
+        <xacro:inertial_cylinder mass="${wheel_mass}" length="${wheel_thickness}" radius="${wheel_radius}">
+            <origin xyz="0 0 0" rpy="0 0 0"/>
+        </xacro:inertial_cylinder>
+    </link>
+    <gazebo reference="left_upper_wheel">
+        <material>Gazebo/Blue</material>
+    </gazebo> -->
+    <!-- Right wheel link -->
+    <joint name="right_wheel_joint" type="continuous">
+        <parent link="base_link"/>
+        <child link="right_wheel"/>
         <origin xyz="${-wheel_offset_x} ${-wheel_offset_y} 0" rpy="${pi/2} 0 0"/>
         <axis xyz="0 0 -1"/>
     </joint>
-    <link name="rear_right_wheel">
-        <visual>
-            <geometry>
-                <cylinder radius="${wheel_radius}" length="${wheel_thickness}"/>
-            </geometry>
-            <material name="blue"/>
-        </visual>
-        <collision>
-            <geometry>
-                <sphere radius="${wheel_radius}"/>
-            </geometry>
-        </collision>
-        <xacro:inertial_cylinder mass="${wheel_mass}" length="${wheel_thickness}" radius="${wheel_radius}">
-            <origin xyz="0 0 0" rpy="0 0 0"/>
-        </xacro:inertial_cylinder>
-    </link>
-    <gazebo reference="rear_right_wheel">
-        <material>Gazebo/Blue</material>
-        <mu1 value="1.0"/>
-        <mu2 value="0.5"/>
-    </gazebo>
-    <!-- FRONT RIGHT WHEEL LINK -->
-    <joint name="front_right_wheel_joint" type="continuous">
-        <parent link="base_link"/>
-        <child link="front_right_wheel"/>
+    <link name="right_wheel">
+        <visual>
+            <geometry>
+                <cylinder radius="${wheel_radius}" length="${wheel_thickness}"/>
+            </geometry>
+            <material name="blue"/>
+        </visual>
+        <collision>
+            <geometry>
+                <sphere radius="${wheel_radius}"/>
+            </geometry>
+        </collision>
+        <xacro:inertial_cylinder mass="${wheel_mass}" length="${wheel_thickness}" radius="${wheel_radius}">
+            <origin xyz="0 0 0" rpy="0 0 0"/>
+        </xacro:inertial_cylinder>
+    </link>
+    <gazebo reference="right_wheel">
+        <material>Gazebo/Blue</material>
+    </gazebo>
+    <!-- <joint name="right_upper_wheel_joint" type="continuous">
+        <parent link="base_link"/>
+        <child link="right_upper_wheel"/>
         <origin xyz="${wheel_offset_x} ${-wheel_offset_y} 0" rpy="${pi/2} 0 0"/>
         <axis xyz="0 0 -1"/>
     </joint>
-    <link name="front_right_wheel">
-        <visual>
-            <geometry>
-                <cylinder radius="${wheel_radius}" length="${wheel_thickness}"/>
-            </geometry>
-            <material name="blue"/>
-        </visual>
-        <collision>
-            <geometry>
-                <sphere radius="${wheel_radius}"/>
-            </geometry>
-        </collision>
-        <xacro:inertial_cylinder mass="${wheel_mass}" length="${wheel_thickness}" radius="${wheel_radius}">
-            <origin xyz="0 0 0" rpy="0 0 0"/>
-        </xacro:inertial_cylinder>
-    </link>
-    <gazebo reference="front_right_wheel">
-        <material>Gazebo/Blue</material>
-        <mu1 value="1.0"/>
-        <mu2 value="0.5"/>
+    <link name="right_upper_wheel">
+        <visual>
+            <geometry>
+                <cylinder radius="${wheel_radius}" length="${wheel_thickness}"/>
+            </geometry>
+            <material name="blue"/>
+        </visual>
+        <collision>
+            <geometry>
+                <sphere radius="${wheel_radius}"/>
+            </geometry>
+        </collision>
+        <xacro:inertial_cylinder mass="${wheel_mass}" length="${wheel_thickness}" radius="${wheel_radius}">
+            <origin xyz="0 0 0" rpy="0 0 0"/>
+        </xacro:inertial_cylinder>
+    </link>
+    <gazebo reference="right_upper_wheel">
+        <material>Gazebo/Blue</material>
+    </gazebo> -->
+    <!-- Caster wheel link -->
+    <joint name="caster_wheel_joint" type="fixed">
+        <parent link="base_link"/>
+        <child link="caster_wheel"/>
+        <origin xyz="${caster_wheel_offset_x} 0 ${caster_wheel_offset_z}"/>
+    </joint>
+    <link name="caster_wheel">
+        <visual>
+            <geometry>
+                <sphere radius="${caster_wheel_radius}"/>1
+            </geometry>
+            <material name="blue"/>
+        </visual>
+        <collision>
+            <geometry>
+                <sphere radius="${caster_wheel_radius}"/>
+            </geometry>
+        </collision>
+        <xacro:inertial_sphere mass="${caster_wheel_mass}" radius="${caster_wheel_radius}">
+            <origin xyz="0 0 0" rpy="0 0 0"/>
+        </xacro:inertial_sphere>
+    </link>
+    <gazebo reference="caster_wheel">
+        <material>Gazebo/Blue</material>
+        <mu1 value="0.001"/>
+        <mu2 value="0.001"/>
     </gazebo>
 </robot>
