Commit message: i

File: description/robot.urdf.xacro (robot description, xacro)
@@ -1,10 +1,10 @@
 <?xml version="1.0"?>
 <robot xmlns:xacro="http://www.ros.org/wiki/xacro"  name="robot">
-    <xacro:arg name="use_ros2_control" default="true"></xacro:arg>
+    <xacro:arg name="use_ros2_control" default="true"/>
     <xacro:include filename="robot_core.xacro" />
-    <xacro:if value="${arg use_ros2_control}">
+    <xacro:if value="$(arg use_ros2_control)">
         <xacro:include filename="ros2_control.xacro" />
     </xacro:if>
-    <xacro:unless value="${arg use_ros2_control}">
+    <xacro:unless value="$(arg use_ros2_control)">
         <xacro:include filename="gazebo_control.xacro" />
     </xacro:unless>

File: description/robot_core.xacro (robot description, xacro)
@@ -2,4 +2,18 @@
 <robot xmlns:xacro="http://www.ros.org/wiki/xacro">
     <xacro:include filename="inertial_macros.xacro" />
+    <xacro:property name="chassis_length" value="0.22"/>
+    <xacro:property name="chassis_width" value="0.15"/>
+    <xacro:property name="chassis_height" value="0.095"/>
+    <xacro:property name="chassis_mass" value="1.0"/>
+    <xacro:property name="wheel_radius" value="0.048"/>
+    <xacro:property name="wheel_thickness" value="0.026"/>
+    <xacro:property name="wheel_mass" value="0.05"/>
+    <xacro:property name="wheel_offset_x" value="0.073"/>
+    <xacro:property name="wheel_offset_y" value="0.1"/>
+    <xacro:property name="wheel_offset_z" value="0.01"/>
+    <xacro:property name="caster_wheel_radius" value="0.048"/>
+    <xacro:property name="caster_wheel_mass" value="0.01"/>
+    <xacro:property name="caster_wheel_offset_x" value="0.075"/>
+    <xacro:property name="caster_wheel_offset_z" value="${wheel_offset_z - wheel_radius + caster_wheel_radius}"/>
     <material name="white">
         <color rgba="1 1 1 1"/>
@@ -40,5 +54,5 @@
             </geometry>
         </collision>
-        <xacro:inertial_box mass="0.5" x="0.24" y="16" z="0.1">
+        <xacro:inertial_box mass="2.0" x="0.24" y="16" z="0.1">
             <origin xyz="0.12 0 0.05" rpy="0 0 0"/>
         </xacro:inertial_box>
@@ -63,8 +77,8 @@
         <collision>
             <geometry>
-                <cylinder radius="0.048" length="0.036"/>
+                <sphere radius="0.048"/>
             </geometry>
         </collision>
-        <xacro:inertial_cylinder mass="0.1" length="0.036" radius="0.048">
+        <xacro:inertial_cylinder mass="0.02" length="0.036" radius="0.048">
             <origin xyz="0 0 0" rpy="0 0 0"/>
         </xacro:inertial_cylinder>
@@ -89,8 +103,8 @@
         <collision>
             <geometry>
-                <cylinder radius="0.048" length="0.036"/>
+                <sphere radius="0.048"/>
             </geometry>
         </collision>
-        <xacro:inertial_cylinder mass="0.1" length="0.036" radius="0.048">
+        <xacro:inertial_cylinder mass="0.02" length="0.036" radius="0.048">
             <origin xyz="0 0 0" rpy="0 0 0"/>
         </xacro:inertial_cylinder>
@@ -104,4 +118,5 @@
         <child link="caster_wheel"/>
         <origin xyz="0.24 0 0"/>
+        <axis xyz="1 1 1"/>
     </joint>
     <link name="caster_wheel">
@@ -117,5 +132,5 @@
             </geometry>
         </collision>
-        <xacro:inertial_sphere mass="0.1" radius="0.048">
+        <xacro:inertial_sphere mass="0.02" radius="0.048">
             <origin xyz="0 0 0" rpy="0 0 0"/>
         </xacro:inertial_sphere>

Commit message: i

File: description/robot.urdf.xacro (robot description, xacro)
@@ -9,4 +9,6 @@
         </xacro:if>
         <xacro:unless value="$(arg use_sim)">
+            <!-- <xacro:include filename="$(find crab_bot)/description/diffbot.ros2_control.xacro" />
+            <xacro:diffbot_ros2_control name="DiffBot" prefix="" /> -->
             <xacro:include filename="ros2_control.hardware.xacro" />
         </xacro:unless>

File: description/ros2_control.hardware.xacro (robot description, xacro)
@@ -1,13 +1,14 @@
 <?xml version="1.0"?>
-<robot xmlns:xacro="http://www.ros.org/wiki/xacro" >
-    <ros2_control name="Real_Robot" type="system">
+<robot xmlns:xacro="http://www.ros.org/wiki/xacro">
+    <ros2_control name="DiffBot" type="system">
         <hardware>
             <plugin>diffdrive_arduino/DiffDriveArduinoHardware</plugin>
-            <param name="left_wheel_name">rear_left_wheel_joint</param>
-            <param name="right_wheel_name">rear_right_wheel_joint</param>
             <param name="front_left_wheel_name">front_left_wheel_joint</param>
+            <param name="rear_left_wheel_name">rear_left_wheel_joint</param>
             <param name="front_right_wheel_name">front_right_wheel_joint</param>
+            <param name="rear_right_wheel_name">rear_right_wheel_joint</param>
             <param name="loop_rate">30</param>
-            <param name="device">/dev/ttyUSB0</param>
+            <!-- <param name="device">/dev/agv-driver</param> -->
+            <param name="device">/dev/cp2104</param>
             <param name="baud_rate">115200</param>
             <param name="timeout_ms">1000</param>
@@ -18,33 +19,21 @@
             <param name="pid_o">50</param>
         </hardware>
-        <joint name="rear_left_wheel_joint" >
-            <command_interface name="velocity">
-                <param name="min">-10</param>
-                <param name="max">10</param>
-            </command_interface>
+        <joint name="rear_left_wheel_joint">
+            <command_interface name="velocity"/>
             <state_interface name="position"/>
             <state_interface name="velocity"/>
         </joint>
-        <joint name="front_left_wheel_joint" >
-            <command_interface name="velocity">
-                <param name="min">-10</param>
-                <param name="max">10</param>
-            </command_interface>
+        <joint name="front_left_wheel_joint">
+            <command_interface name="velocity"/>
             <state_interface name="position"/>
             <state_interface name="velocity"/>
         </joint>
-        <joint name="rear_right_wheel_joint" >
-            <command_interface name="velocity">
-                <param name="min">-10</param>
-                <param name="max">10</param>
-            </command_interface>
+        <joint name="rear_right_wheel_joint">
+            <command_interface name="velocity"/>
             <state_interface name="position"/>
             <state_interface name="velocity"/>
         </joint>
-        <joint name="front_right_wheel_joint" >
-            <command_interface name="velocity">
-                <param name="min">-10</param>
-                <param name="max">10</param>
-            </command_interface>
+        <joint name="front_right_wheel_joint">
+            <command_interface name="velocity"/>
             <state_interface name="position"/>
             <state_interface name="velocity"/>
