Commit message: i

File: description/robot_core.xacro (robot description, xacro)
@@ -41,4 +41,7 @@
         </xacro:inertial_box>
     </link>
+    <gazebo reference="chassis">
+        <material>Gazebo/White</material>
+    </gazebo>
     <!-- Left wheel link -->
     <joint name="left_wheel_joint" type="continuous">
@@ -64,4 +67,7 @@
         </xacro:inertial_cylinder>
     </link>
+    <gazebo reference="left_wheel">
+        <material>Gazebo/Blue</material>
+    </gazebo>
     <!-- Right wheel link -->
     <joint name="right_wheel_joint" type="continuous">
@@ -87,4 +93,7 @@
         </xacro:inertial_cylinder>
     </link>
+    <gazebo reference="right_wheel">
+        <material>Gazebo/Blue</material>
+    </gazebo>
     <!-- Caster wheel link -->
     <joint name="caster_wheel_joint" type="fixed">
@@ -109,3 +118,6 @@
         </xacro:inertial_sphere>
     </link>
+    <gazebo reference="caster_wheel">
+        <material>Gazebo/Blue</material>
+    </gazebo>
 </robot>

Commit message: i

File: description/robot_core.xacro (robot description, xacro)
@@ -2,18 +2,18 @@
 <robot xmlns:xacro="http://www.ros.org/wiki/xacro">
     <xacro:include filename="inertial_macros.xacro" />
-    <xacro:property name="chassis_length" value="0.22"/>
+    <xacro:property name="chassis_length" value="0.225"/>
     <xacro:property name="chassis_width" value="0.15"/>
-    <xacro:property name="chassis_height" value="0.095"/>
-    <xacro:property name="chassis_mass" value="1.0"/>
+    <xacro:property name="chassis_height" value="0.0975"/>
+    <xacro:property name="chassis_mass" value="4.0"/>
     <xacro:property name="wheel_radius" value="0.048"/>
-    <xacro:property name="wheel_thickness" value="0.026"/>
+    <xacro:property name="wheel_thickness" value="0.036"/>
     <xacro:property name="wheel_mass" value="0.05"/>
     <xacro:property name="wheel_offset_x" value="0.073"/>
     <xacro:property name="wheel_offset_y" value="0.1"/>
-    <xacro:property name="wheel_offset_z" value="0.01"/>
-    <xacro:property name="caster_wheel_radius" value="0.048"/>
+    <xacro:property name="wheel_offset_z" value="0.02"/>
+    <xacro:property name="caster_wheel_radius" value="0.01"/>
     <xacro:property name="caster_wheel_mass" value="0.01"/>
-    <xacro:property name="caster_wheel_offset_x" value="0.075"/>
-    <xacro:property name="caster_wheel_offset_z" value="${wheel_offset_z - wheel_radius + caster_wheel_radius}"/>
+    <xacro:property name="caster_wheel_offset_x" value="0.073"/>
+    <xacro:property name="caster_wheel_offset_z" value="${-wheel_radius + caster_wheel_radius}"/>
     <material name="white">
         <color rgba="1 1 1 1"/>
@@ -34,26 +34,37 @@
     <link name="base_link">
     </link>
+    <!-- BASE_FOOTPRINT LINK -->
+    <joint name="base_footprint_joint" type="fixed">
+        <parent link="base_link"/>
+        <child link="base_footprint"/>
+        <origin xyz="0 0 0" rpy="0 0 0"/>
+    </joint>
+    <link name="base_footprint">
+    </link>
     <!-- Chassis link -->
     <joint name="chassis_joint" type="fixed">
         <parent link="base_link"/>
         <child link="chassis"/>
-        <origin xyz="-0.047 0 0"/>
+        <origin xyz="${-chassis_length/2} 0 0"/>
     </joint>
     <link name="chassis">
+        <!-- chassis visual -->
         <visual>
-            <origin xyz="0.12 0 0.05"/>
+            <origin xyz="${chassis_length/2} 0 ${chassis_height/2}"/>
             <geometry>
-                <box size="0.24 0.16 0.1"/>
+                <box size="${chassis_length} ${chassis_width} ${chassis_height}"/>
             </geometry>
             <material name="white"/>
         </visual>
+        <!-- chassis interact -->
         <collision>
-            <origin xyz="0.12 0 0.05"/>
+            <origin xyz="${chassis_length/2} 0 ${chassis_height/2}"/>
             <geometry>
-                <box size="0.24 0.16 0.1"/>
+                <box size="${chassis_length} ${chassis_width} ${chassis_height}"/>
             </geometry>
         </collision>
-        <xacro:inertial_box mass="2.0" x="0.24" y="16" z="0.1">
-            <origin xyz="0.12 0 0.05" rpy="0 0 0"/>
+        <!-- chassis phisical -->
+        <xacro:inertial_box mass="2.0" x="${chassis_length}" y="${chassis_width}" z="${chassis_height}">
+            <origin xyz="${chassis_length/2} 0 ${chassis_height/2}" rpy="0 0 0"/>
         </xacro:inertial_box>
     </link>
@@ -65,5 +76,5 @@
         <parent link="base_link"/>
         <child link="left_wheel"/>
-        <origin xyz="0 0.1 0" rpy="-${pi/2} 0 0"/>
+        <origin xyz="${-wheel_offset_x} ${wheel_offset_y} 0" rpy="-${pi/2} 0 0"/>
         <axis xyz="0 0 1"/>
     </joint>
@@ -71,5 +82,5 @@
         <visual>
             <geometry>
-                <cylinder radius="0.048" length="0.036"/>
+                <cylinder radius="${wheel_radius}" length="${wheel_thickness}"/>
             </geometry>
             <material name="blue"/>
@@ -77,8 +88,8 @@
         <collision>
             <geometry>
-                <sphere radius="0.048"/>
+                <sphere radius="${wheel_radius}"/>
             </geometry>
         </collision>
-        <xacro:inertial_cylinder mass="0.02" length="0.036" radius="0.048">
+        <xacro:inertial_cylinder mass="${wheel_mass}" length="${wheel_thickness}" radius="${wheel_radius}">
             <origin xyz="0 0 0" rpy="0 0 0"/>
         </xacro:inertial_cylinder>
@@ -91,5 +102,5 @@
         <parent link="base_link"/>
         <child link="right_wheel"/>
-        <origin xyz="0 -0.1 0" rpy="${pi/2} 0 0"/>
+        <origin xyz="${-wheel_offset_x} ${-wheel_offset_y} 0" rpy="${pi/2} 0 0"/>
         <axis xyz="0 0 -1"/>
     </joint>
@@ -97,5 +108,5 @@
         <visual>
             <geometry>
-                <cylinder radius="0.048" length="0.036"/>
+                <cylinder radius="${wheel_radius}" length="${wheel_thickness}"/>
             </geometry>
             <material name="blue"/>
@@ -103,8 +114,8 @@
         <collision>
             <geometry>
-                <sphere radius="0.048"/>
+                <sphere radius="${wheel_radius}"/>
             </geometry>
         </collision>
-        <xacro:inertial_cylinder mass="0.02" length="0.036" radius="0.048">
+        <xacro:inertial_cylinder mass="${wheel_mass}" length="${wheel_thickness}" radius="${wheel_radius}">
             <origin xyz="0 0 0" rpy="0 0 0"/>
         </xacro:inertial_cylinder>
@@ -115,13 +126,12 @@
     <!-- Caster wheel link -->
     <joint name="caster_wheel_joint" type="fixed">
-        <parent link="chassis"/>
+        <parent link="base_link"/>
         <child link="caster_wheel"/>
-        <origin xyz="0.24 0 0"/>
-        <axis xyz="1 1 1"/>
+        <origin xyz="${caster_wheel_offset_x} 0 ${caster_wheel_offset_z}"/>
     </joint>
     <link name="caster_wheel">
         <visual>
             <geometry>
-                <sphere radius="0.048"/>
+                <sphere radius="0.01"/>1
             </geometry>
             <material name="blue"/>
@@ -129,8 +139,8 @@
         <collision>
             <geometry>
-                <sphere radius="0.048"/>
+                <sphere radius="0.01"/>
             </geometry>
         </collision>
-        <xacro:inertial_sphere mass="0.02" radius="0.048">
+        <xacro:inertial_sphere mass="0.02" radius="0.01">
             <origin xyz="0 0 0" rpy="0 0 0"/>
         </xacro:inertial_sphere>

Commit message: i

File: description/robot_core.xacro (robot description, xacro)
@@ -73,9 +73,10 @@
         <parent link="base_link"/>
         <child link="rear_left_wheel"/>
-        <origin xyz="${-wheel_offset_x} ${wheel_offset_y} 0" rpy="-${pi/2} 0 0"/>
-        <axis xyz="0 0 1"/>
+        <origin xyz="${-wheel_offset_x} ${wheel_offset_y} 0" rpy="0 0 0"/>
+        <axis xyz="0 1 0" rpy="0 0 0"/>
     </joint>
     <link name="rear_left_wheel">
         <visual>
+            <origin xyz="0 0 0" rpy="${pi/2} 0 0" />
             <geometry>
                 <cylinder radius="${wheel_radius}" length="${wheel_thickness}"/>
@@ -84,6 +85,7 @@
         </visual>
         <collision>
+            <origin xyz="0 0 0" rpy="${pi/2} 0 0" />
             <geometry>
-                <sphere radius="${wheel_radius}"/>
+                <cylinder radius="${wheel_radius}" length="${wheel_thickness}"/>
             </geometry>
         </collision>
@@ -95,5 +97,6 @@
         <material>Gazebo/Blue</material>
         <mu1 value="1.0"/>
-        <mu2 value="0.5"/>
+        <mu2 value="0.1"/>
+        <fdir1>1 0 0</fdir1>
     </gazebo>
     <!-- FRONT LEFT WHEEL LINK -->
@@ -101,9 +104,10 @@
         <parent link="base_link"/>
         <child link="front_left_wheel"/>
-        <origin xyz="${wheel_offset_x} ${wheel_offset_y} 0" rpy="-${pi/2} 0 0"/>
-        <axis xyz="0 0 1"/>
+        <origin xyz="${wheel_offset_x} ${wheel_offset_y} 0" rpy="0 0 0"/>
+        <axis xyz="0 1 0" rpy="0 0 0"/>
     </joint>
     <link name="front_left_wheel">
         <visual>
+            <origin xyz="0 0 0" rpy="${pi/2} 0 0" />
             <geometry>
                 <cylinder radius="${wheel_radius}" length="${wheel_thickness}"/>
@@ -112,6 +116,7 @@
         </visual>
         <collision>
+            <origin xyz="0 0 0" rpy="${pi/2} 0 0" />
             <geometry>
-                <sphere radius="${wheel_radius}"/>
+                <cylinder radius="${wheel_radius}" length="${wheel_thickness}"/>
             </geometry>
         </collision>
@@ -123,5 +128,6 @@
         <material>Gazebo/Blue</material>
         <mu1 value="1.0"/>
-        <mu2 value="0.5"/>
+        <mu2 value="0.1"/>
+        <fdir1>1 0 0</fdir1>
     </gazebo>
     <!-- REAR RIGHT WHEEL LINK -->
@@ -129,9 +135,10 @@
         <parent link="base_link"/>
         <child link="rear_right_wheel"/>
-        <origin xyz="${-wheel_offset_x} ${-wheel_offset_y} 0" rpy="${pi/2} 0 0"/>
-        <axis xyz="0 0 -1"/>
+        <origin xyz="${-wheel_offset_x} ${-wheel_offset_y} 0" rpy="0 0 0"/>
+        <axis xyz="0 1 0" rpy="0 0 0"/>
     </joint>
     <link name="rear_right_wheel">
         <visual>
+            <origin xyz="0 0 0" rpy="${pi/2} 0 0" />
             <geometry>
                 <cylinder radius="${wheel_radius}" length="${wheel_thickness}"/>
@@ -140,6 +147,7 @@
         </visual>
         <collision>
+            <origin xyz="0 0 0" rpy="${pi/2} 0 0" />
             <geometry>
-                <sphere radius="${wheel_radius}"/>
+                <cylinder radius="${wheel_radius}" length="${wheel_thickness}"/>
             </geometry>
         </collision>
@@ -151,5 +159,6 @@
         <material>Gazebo/Blue</material>
         <mu1 value="1.0"/>
-        <mu2 value="0.5"/>
+        <mu2 value="0.1"/>
+        <fdir1>1 0 0</fdir1>
     </gazebo>
     <!-- FRONT RIGHT WHEEL LINK -->
@@ -157,9 +166,10 @@
         <parent link="base_link"/>
         <child link="front_right_wheel"/>
-        <origin xyz="${wheel_offset_x} ${-wheel_offset_y} 0" rpy="${pi/2} 0 0"/>
-        <axis xyz="0 0 -1"/>
+        <origin xyz="${wheel_offset_x} ${-wheel_offset_y} 0" rpy="0 0 0"/>
+        <axis xyz="0 1 0" rpy="0 0 0"/>
     </joint>
     <link name="front_right_wheel">
         <visual>
+            <origin xyz="0 0 0" rpy="${pi/2} 0 0" />
             <geometry>
                 <cylinder radius="${wheel_radius}" length="${wheel_thickness}"/>
@@ -168,6 +178,7 @@
         </visual>
         <collision>
+            <origin xyz="0 0 0" rpy="${pi/2} 0 0" />
             <geometry>
-                <sphere radius="${wheel_radius}"/>
+                <cylinder radius="${wheel_radius}" length="${wheel_thickness}"/>
             </geometry>
         </collision>
@@ -179,5 +190,6 @@
         <material>Gazebo/Blue</material>
         <mu1 value="1.0"/>
-        <mu2 value="0.5"/>
+        <mu2 value="0.1"/>
+        <fdir1>1 0 0</fdir1>
     </gazebo>
 </robot>

Commit message: i

File: description/robot_core.xacro (robot description, xacro)
@@ -62,5 +62,5 @@
         </collision>
         <!-- chassis phisical -->
-        <xacro:inertial_box mass="0.5" x="${chassis_length}" y="${chassis_width}" z="${chassis_height}">
+        <xacro:inertial_box mass="${chassis_mass}" x="${chassis_length}" y="${chassis_width}" z="${chassis_height}">
             <origin xyz="0 0 ${chassis_height/2}" rpy="0 0 0"/>
         </xacro:inertial_box>
@@ -81,4 +81,5 @@
             <geometry>
                 <cylinder radius="${wheel_radius}" length="${wheel_thickness}"/>
+                <!-- <mesh filename="package://description/meshes/Wheel96.STL" /> -->
             </geometry>
             <material name="blue"/>
@@ -87,5 +88,5 @@
             <origin xyz="0 0 0" rpy="${pi/2} 0 0" />
             <geometry>
-                <cylinder radius="${wheel_radius}" length="${wheel_thickness}"/>
+                <cylinder radius="${wheel_radius}" length="${wheel_thickness/4}"/>
             </geometry>
         </collision>
@@ -118,5 +119,5 @@
             <origin xyz="0 0 0" rpy="${pi/2} 0 0" />
             <geometry>
-                <cylinder radius="${wheel_radius}" length="${wheel_thickness}"/>
+                <cylinder radius="${wheel_radius}" length="${wheel_thickness/4}"/>
             </geometry>
         </collision>
@@ -149,5 +150,5 @@
             <origin xyz="0 0 0" rpy="${pi/2} 0 0" />
             <geometry>
-                <cylinder radius="${wheel_radius}" length="${wheel_thickness}"/>
+                <cylinder radius="${wheel_radius}" length="${wheel_thickness/4}"/>
             </geometry>
         </collision>
@@ -180,5 +181,5 @@
             <origin xyz="0 0 0" rpy="${pi/2} 0 0" />
             <geometry>
-                <cylinder radius="${wheel_radius}" length="${wheel_thickness}"/>
+                <cylinder radius="${wheel_radius}" length="${wheel_thickness/4}"/>
             </geometry>
         </collision>
