Commit message: i

File: crabbot_description/accessories/dept_camera.xacro (robot description, xacro)
@@ -6,5 +6,5 @@
             <origin xyz="0 0 0" rpy="0 0 0"/>
             <geometry>
-            <box size="0.015 0.130 0.022"/>
+            <box size="0.025 0.095 0.025"/>
             </geometry>
         </visual>
@@ -12,5 +12,5 @@
             <origin xyz="0 0 0" rpy="0 0 0"/>
             <geometry>
-            <box size="0.015 0.130 0.022"/>
+            <box size="0.025 0.095 0.025"/>
             </geometry>
         </collision>

File: crabbot_description/robot.urdf.xacro (robot description, xacro)
@@ -4,6 +4,6 @@
     <xacro:include filename="ros2_control.xacro" />
     <xacro:include filename="accessories/lidar.xacro" />
-    <xacro:include filename="accessories/camera.xacro" />
-    <!-- <xacro:include filename="accessories/dept_camera.xacro" /> -->
+    <!-- <xacro:include filename="accessories/camera.xacro" /> -->
+    <xacro:include filename="accessories/dept_camera.xacro" />
     <!-- <xacro:include filename="accessories/imu.xacro" /> -->
 </robot>

Commit message: i

File: crabbot_description/accessories/dept_camera.xacro (robot description, xacro)
@@ -35,7 +35,7 @@
     </joint>
     <!-- Gazebo Plugin -->
-    <!-- <gazebo reference="camera_link">
+    <gazebo reference="camera_link">
         <material>Gazebo/Blue</material>
-        <sensor name="depth_camera" type="depth">
+        <sensor name="camera" type="depth">
             <visualize>true</visualize>
             <update_rate>30.0</update_rate>
@@ -70,5 +70,23 @@
                 <hackBaseline>0</hackBaseline>
             </plugin>
+            <plugin name="camera_controller" filename="libgazebo_ros_camera.so">
+                <baseline>0.2</baseline>
+                <alwaysOn>true</alwaysOn>
+                <updateRate>0.0</updateRate>
+                <frame_name>camera_depth_frame</frame_name>
+                <pointCloudCutoff>0.5</pointCloudCutoff>
+                <pointCloudCutoffMax>3.0</pointCloudCutoffMax>
+                <distortionK1>0</distortionK1>
+                <distortionK2>0</distortionK2>
+                <distortionK3>0</distortionK3>
+                <distortionT1>0</distortionT1>
+                <distortionT2>0</distortionT2>
+                <CxPrime>0</CxPrime>
+                <Cx>0</Cx>
+                <Cy>0</Cy>
+                <focalLength>0</focalLength>
+                <hackBaseline>0</hackBaseline>
+            </plugin>
         </sensor>
-    </gazebo> -->
+    </gazebo>
 </robot>

File: crabbot_description/accessories/imu.xacro (robot description, xacro)
@@ -23,5 +23,5 @@
     </joint>
     <!--  -->
-    <!-- <gazebo reference="imu_link">
+    <gazebo reference="imu_link">
         <sensor name="imu_sensor" type="imu">
             <plugin filename="libgazebo_ros_imu_sensor.so" name="imu_plugin">
@@ -90,4 +90,4 @@
             </imu>
         </sensor>
-    </gazebo> -->
+    </gazebo>
 </robot>

File: crabbot_description/accessories/lidar.xacro (robot description, xacro)
@@ -63,5 +63,5 @@
         </sensor>
     </gazebo>
-    <!-- <joint name="laser_joint" type="fixed">
+    <joint name="laser_joint" type="fixed">
         <parent link="base_link"/>
         <child link="laser_frame"/>
@@ -113,4 +113,4 @@
             </plugin>
         </sensor>
-    </gazebo> -->
+    </gazebo>
 </robot>

File: crabbot_description/robot.2wd.urdf.xacro (robot description, xacro)
@@ -6,4 +6,4 @@
     <!-- <xacro:include filename="accessories/camera.xacro" /> -->
     <xacro:include filename="accessories/dept_camera.xacro" />
-    <!-- <xacro:include filename="accessories/imu.xacro" /> -->
+    <xacro:include filename="accessories/imu.xacro" />
 </robot>
